File: PCB_4.1x4.1/circuito_tesi.sch (EAGLE design)
At the start: 43 parts, among them IC1 SCD41-D-R2, IC2 TPS60120PWPR, IC3 TPS78918DBVR, Q1 BSS138, Q2 BSS138, Q3 BSS138, Q4 BSS138, U1 TSV912IDT, U2 SGP30, U3 MICS-6814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

Commit message: PCB prima prova
Parts:
- added C1, C12, C13: CL05A106MP5NUNC, Condens_10uF:CL05A106MP5NUNC
- added C2, C3, C5: GRM033R61A225KE47D, Condens_2.2uF:GRM033R61A225KE47D
- added C4: CL05A226MQ5N6J8, Condens_22uF:CL05A226MQ5N6J8
- added C6: GRM033R60J105MEA2D, Condens_1uF:GRM033R60J105MEA2D
- added R18: ERA6VEB8200V, Res_820_0p25W:ERA6VEB8200V
Connections:
- new net N$12: C2.1, IC2.C1-
- new net N$14: C3.2, IC2.C2+
- new net N$18: C3.1, IC2.C2-
- new net N$19: IC2.FB, IC2.OUT_1
- new net N$20: C6.2, U8.CXN
- new net N$22: C6.1, U8.CXP
- new net N$24: R18.1, U8.!SHDN
- new net N$7: C2.2, IC2.C1+
- net 3.3: now also C13.1, C4.2, C5.2, Q4.G, R16.2, R18.2; no longer IC1.VDD, IC1.VDDH
- net 5V: now also C12.1, IC1.VDD, IC1.VDDH; no longer Q4.G, R16.2
- net GND: now also C1.2, C12.2, C13.2, C4.1, C5.1, U5.GND
- net N$1: now also IC1.SDA
- net N$15: now also U5.P0.05/AIN3; no longer U5.P0.03/AIN1
- net N$17: now also U5.P0.03/AIN1; no longer U5.P0.05/AIN3
- net N$21: now also U5.P0.25; no longer U5.P0.13
- net N$3: now also IC1.SCL
- net SCL: now also U5.P0.26; no longer IC1.SCL, U5.P0.12
- net SDA: now also U5.P0.27; no longer IC1.SDA, U5.P0.11
- net VDD: now also C1.1
Other:
- moved on the sheet: LED2, Q3, Q4, R14, R15, R16, R17
