File: PCB_SecondaVersione/circuito_tesi.brd (EAGLE design)
At the start: 100 x 80 mm, 50 parts, among them IC1 SCD41-D-R2, Q1 BSS138, Q2 BSS138, Q3 BSS138, Q4 BSS138, U3 MICS-6814, U6 BME280, U7 LIS3DH

Commit message: Aggiunti case 0402
Parts:
- removed C10_10: CL21A226MOQNNNE, Cond_22uF_0805:CAPC2012X135N
- removed C1_0.1, C2_0.1, C7_0.01, C8_0.02, C9_0.1: CL21B104KCFNNNE, Cond_100nF_0805:CAPC2012X140N
- removed C3_2.2, C4_470P: CL21A475KAQNNNE, Cond_4.7uF_0805:CAPC2012X140N
- removed C5_1, C6_2: CL21B105KAFNNNE, Cond_1uF_0805:CAPC2012X140N
- added C1, C10, C11, C12, C13, C2, C3, C4, C5, C6, C7, C8, C9: C0402H102J5GACTU, Condensatore_case_0402:CAPC1005X55N
- added PROGRAMMER: BG306-04-A-1-0400-X-X_REVD, Connet_6_BG306-04-A-1-0400-X-X_REVD:GCT_BG306-04-A-1-0400-X-X_REVD
- added R19, R20: 8-1879333-9, Resistenza_case_0402:RESC1005X35N
- added Y1: ECS-.327-9-16-TR, Crystal-ECS-.327-9-16-TR:XTAL_ECS-.327-9-16-TR
- R1, R10, R2, R3, R4, R5, R6, R7, R8, R9: value RNCP0805FTD10K0 -> 8-1879333-9; device Res_10K_0p25W:RESC2012X60N -> Resistenza_case_0402:RESC1005X35N
- R11: value RP73PF2A130RBTDF -> 8-1879333-9; device Res_130_0p25:RESC2012X65N -> Resistenza_case_0402:RESC1005X35N
- R12: value ERA6VEB8200V -> 8-1879333-9; device Res_820_0p25W:RES_ERA6VEB8200V -> Resistenza_case_0402:RESC1005X35N
- R13, R14: value RMCF0603FT5M10 -> 8-1879333-9; device Res_5.1MOHM:RESC1508X55N -> Resistenza_case_0402:RESC1005X35N
- R15, R16: value RMCF0603FT10M0 -> 8-1879333-9; device Res_10MOHM_2:RESC1508X55N -> Resistenza_case_0402:RESC1005X35N
- R17: value ERJ-PB6D5101V -> 8-1879333-9; device Res_5.1K_0805:RESC2012X70N -> Resistenza_case_0402:RESC1005X35N
- R18: value ERJ-PB6B3300V -> 8-1879333-9; device Res_330_0805:RESC2012X70N -> Resistenza_case_0402:RESC1005X35N
- SPS30: value (none) -> BG306-05-A-1-0400-X-X_REVD; device con-lstb:MA05-1 -> Connet_5_BG306-05-A-1-0400-X-X_REVD:GCT_BG306-05-A-1-0400-X-X_REVD
- moved R16 244.5 mm to (-104.0, -149.0)
- moved R15 244.3 mm to (-104.0, -146.0)
- moved R14 234.3 mm to (-104.0, -143.0)
- moved R13 233.6 mm to (-104.0, -140.0)
- moved R10 214.9 mm to (-104.0, -131.0)
- moved R11 213.8 mm to (-104.0, -134.0)
- moved R12 212.6 mm to (-104.0, -137.0)
- moved R9 210.4 mm to (-104.0, -128.0)
- moved R8 206.2 mm to (-104.0, -125.0)
- moved R6 205.1 mm to (-104.0, -119.0)
- moved R5 204.4 mm to (-104.0, -116.0)
- moved R2 204.2 mm to (-104.0, -107.0)
- moved R4 204.0 mm to (-104.0, -113.0)
- moved R3 204.0 mm to (-104.0, -110.0)
- moved R7 202.2 mm to (-104.0, -122.0)
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Connections:
- net N$1 renamed SDA5
- net N$12 renamed SCL18
- net N$16 renamed SDA18
- removed net N$5: Q4.3, R7.1, SPS30.3
- new net AIN4: C9.1, MDBT42Q.5, R19.2, R20.2
- new net N$17: C12.1, MDBT42Q.13, Y1.2
- new net N$18: C13.1, MDBT42Q.14, Y1.1
- new net SCL5: Q4.3, R7.2, SPS30.3
- net 1.8V: now also C10.2, C6.1; no longer C6_2.1, C9_0.1.2
- net 3.3V: now also C11.2, C3.1, PROGRAMMER.1; no longer C10_10.2, C3_2.2.1
- net 5V: now also C2.1, R11.1, R12.1, R7.1; no longer C2_0.1.1, R11.2, R12.2, R7.2
- net AIN1: now also C7.2, R13.1, R15.1; no longer C7_0.01.2, R13.2, R15.2
- net AIN3: now also C8.1; no longer C8_0.02.1
- net GND: now also C1.2, C10.1, C11.1, C12.2, C13.2, C2.2, C3.2, C4.2, C5.2, C6.2, C7.1, C8.2, C9.2, PROGRAMMER.4, R15.2, R20.1; no longer C10_10.1, C1_0.1.2, C2_0.1.2, C3_2.2.2, C4_470P.2, C5_1.2, C6_2.2, C7_0.01.1, C8_0.02.2, C9_0.1.1, R15.1
- net N$11: now also R12.2; no longer R12.1
- net N$13: now also R11.2; no longer R11.1
- net N$14: now also C4.1; no longer C4_470P.1
- net N$8: now also R13.2; no longer R13.1
- net SWDCLK: now also PROGRAMMER.3
- net SWDIO: now also PROGRAMMER.2
- net VDD: now also C1.1, C5.1, R19.1; no longer C1_0.1.1, C5_1.1

Commit message: Posizionamento su PCB
Parts:
- moved C10 289.9 mm to (49.0, 64.0)
- moved C9 269.5 mm to (43.0, 45.0), flipped to the bottom
- moved C11 264.0 mm to (32.0, 42.0)
- moved R18 262.3 mm to (49.0, 58.0)
- moved C13 261.6 mm to (27.0, 38.0)
- moved C12 260.0 mm to (24.0, 41.0)
- moved C5 257.6 mm to (36.0, 45.0), flipped to the bottom
- moved C6 257.6 mm to (33.0, 45.0), flipped to the bottom
- moved R20 254.7 mm to (43.0, 47.0), flipped to the bottom
- moved R19 253.9 mm to (43.0, 49.0), flipped to the bottom
- moved C4 251.1 mm to (28.0, 45.0), flipped to the bottom
- moved C3 247.7 mm to (25.0, 45.0), flipped to the bottom
- moved C7 245.2 mm to (24.0, 34.0), turned to 180 degrees
- moved C2 243.3 mm to (20.0, 45.0), flipped to the bottom
- moved C8 243.2 mm to (24.0, 29.0), turned to 180 degrees
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