File: PCB_SecondaVersione/circuito_tesi.brd (EAGLE design)
At the start: 100 x 80 mm, 57 parts, among them IC1 SCD41-D-R2, Q1 BSS138, Q2 BSS138, Q3 BSS138, Q4 BSS138, U3 MICS-6814, U6 BME280, U7 LIS3DH, Y1 ECS-.327-9-16-TR

Commit message: Inizio board
Parts:
- moved U6 34.5 mm to (58.6, 65.4)
- moved R1 31.4 mm to (65.1, 61.0)
- moved R2 29.8 mm to (61.0, 61.0)
- moved U7 25.5 mm to (58.7, 70.4)
- moved MDBT42Q 21.7 mm to (20.2, 46.8), turned to 90 degrees
- moved SPS30 18.4 mm to (32.0, 64.0), turned to 0 degrees
- moved IC1 18.4 mm to (40.0, 45.5)
- moved PROGRAMMER 16.1 mm to (42.0, 31.0)
- moved R19 15.1 mm to (28.2, 45.9), turned to 270 degrees
- moved C9 13.6 mm to (29.6, 42.5), turned to 270 degrees
- moved C3 12.9 mm to (37.9, 44.8), turned to 180 degrees
- moved R20 12.6 mm to (31.2, 42.5), turned to 90 degrees
- moved R11 11.2 mm to (13.0, 39.0)
- moved C5 9.67 mm to (45.5, 46.8), turned to 270 degrees
- moved OPAMP 9.33 mm to (25.7, 33.3)
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Connections:
- new net BJT: BJT.2, OPAMP.8, R11.1, R12.1
- new net P7: MDBT42Q.7, R17.1
- net 5V: now also BJT.3; no longer OPAMP.8, R11.1, R12.1
Routing:
- net VDD: track 0.00 -> 46.9 mm
- net N$4: track 0.00 -> 45.1 mm
- net N$25: track 0.00 -> 37.2 mm
- net N$2: track 0.00 -> 36.3 mm
- net BJT: track 0.00 -> 35.5 mm
- net N$27: track 0.00 -> 33.0 mm
- net GND: track 0.00 -> 28.2 mm
- net N$10: track 0.00 -> 12.8 mm
- net N$6: track 0.00 -> 11.2 mm
- net N$13: track 0.00 -> 7.61 mm
- net N$7: track 0.00 -> 6.34 mm
- net AIN4: track 0.00 -> 5.73 mm
- net N$17: track 0.00 -> 4.89 mm
- net N$18: track 0.00 -> 4.89 mm
- net AIN1: track 0.00 -> 4.55 mm
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
Commit message: Impostato posizione generale
Parts:
- moved PROGRAMMER 38.9 mm to (15.0, 59.0), turned to 270 degrees
- moved R1 36.4 mm to (31.1, 48.0)
- moved R3 35.1 mm to (35.4, 32.5), turned to 270 degrees
- moved C10 32.2 mm to (46.0, 31.9), turned to 270 degrees
- moved R2 32.0 mm to (31.0, 50.0)
- moved U6 30.8 mm to (40.6, 40.4)
- moved U7 30.0 mm to (40.7, 46.4)
- moved R4 29.6 mm to (40.0, 35.0), turned to 270 degrees
- moved SGP30 28.9 mm to (42.8, 32.3), turned to 180 degrees
- moved Q2 28.3 mm to (45.4, 36.7)
- moved Q1 26.9 mm to (38.4, 33.0)
- moved R7 23.7 mm to (33.0, 52.0)
- moved R5 23.4 mm to (45.6, 33.7)
- moved R8 20.1 mm to (33.0, 54.0)
- moved R6 15.7 mm to (46.1, 39.4), turned to 180 degrees
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Routing:
- net 1.8V: track 1.86 -> 59.6 mm, vias 0 -> 1
- net 5V: track 1.99 -> 50.7 mm, vias 0 -> 2
- net AIN3: track 3.50 -> 30.1 mm
- net AIN1: track 4.55 -> 18.8 mm
- net 3.3V: track 3.69 -> 9.84 mm, vias 0 -> 1
- net GND: track 28.2 -> 31.5 mm
- net AIN4: track 5.73 -> 4.47 mm
- net N$13: track 7.61 -> 6.61 mm
- net N$11: track 4.07 -> 3.07 mm
- net VDD: track 46.9 -> 45.9 mm
- net N$7: track 6.34 -> 5.39 mm
- net N$27: track 33.0 -> 32.2 mm
- net BJT: track 35.5 -> 36.3 mm

Commit message: PCB finita seconda versione
Parts:
- moved R7 8.14 mm to (27.5, 58.0), turned to 90 degrees
- moved R18 6.32 mm to (49.0, 59.0), turned to 270 degrees
- moved R9 5.19 mm to (21.7, 58.0), turned to 270 degrees
- moved R6 2.36 mm to (44.2, 40.8)
- moved U7 2.24 mm to (41.7, 48.4)
- moved R10 2.12 mm to (25.9, 54.3)
- moved R8 1.55 mm to (31.5, 54.4)
- moved R4 1.50 mm to (40.0, 36.5)
- moved R17 1.40 mm to (21.6, 39.7)
- moved BJT 1.30 mm to (18.6, 38.5)
- moved Q4 1.20 mm to (30.1, 57.4), turned to 90 degrees
- moved Q3 0.67 mm to (24.3, 57.3), turned to 90 degrees
- moved C9 0.64 mm to (30.0, 42.0)
- moved R20 0.50 mm to (31.2, 42.0)
- moved IC1 0.41 mm to (40.6, 59.8)
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Connections:
- removed net N$21: LED1.+, MDBT42Q.2
- removed net N$3: R1.1, R2.1
- removed net P7: MDBT42Q.7, R17.1
- new net LED: LED1.+, MDBT42Q.23
- new net P8: MDBT42Q.2, R17.1
- net 3.3V: now also R1.1, R2.1
- net SCL: now also MDBT42Q.19; no longer MDBT42Q.3
- net SDA: now also MDBT42Q.21; no longer MDBT42Q.4
Routing:
- net GND: track 31.5 -> 301.8 mm, vias 0 -> 9
- net 3.3V: track 9.84 -> 134.5 mm, vias 1 -> 5
- net SDA: track 0.00 -> 60.7 mm, vias 0 -> 2
- net SCL: track 0.00 -> 57.7 mm
- net LED: track 0.00 -> 23.8 mm, vias 0 -> 2
- net 5V: track 50.7 -> 64.2 mm
- net AIN4: track 4.47 -> 17.4 mm, vias 0 -> 1
- net SWDIO: track 0.00 -> 10.5 mm
- net SCL5: track 0.00 -> 10.1 mm
- net SWDCLK: track 0.00 -> 6.87 mm
- net SCL18: track 0.05 -> 6.49 mm
- net SDA5: track 0.00 -> 5.99 mm
- net SDA18: track 0.00 -> 5.15 mm
- net VDD: track 45.9 -> 41.2 mm
- net P8: track 0.00 -> 4.40 mm
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