File: PCB_SecondaVersione/circuito_tesi.sch (EAGLE design)
At the start: 52 parts, among them IC1 SCD41-D-R2, IC2 TPS60120PWPR, IC3 TPS78918DBVR, Q1 BSS138, Q2 BSS138, Q3 BSS138, Q4 BSS138, U1 TSV912IDT, U2 SGP30, U3 MICS-6814, U5 317030213, U6 BME280, U7 LIS3DH, U8 MAX682ESA+

Commit message: Sistemato circuito
Parts:
- removed C1, C12: CL05A106MP5NUNC, Condens_10uF:CL05A106MP5NUNC
- removed C10, C11, C6: GRM033R60J105MEA2D, Condens_1uF:GRM033R60J105MEA2D
- removed C2, C3, C5: GRM033R61A225KE47D, Condens_2.2uF:GRM033R61A225KE47D
- removed C4: CL05A226MQ5N6J8, Condens_22uF:CL05A226MQ5N6J8
- removed IC2: TPS60120PWPR, C_P_3.3_TPS60120PWPR:TPS60120PWPR
- removed IC3: TPS78918DBVR, V_REG_1.8_SOT-23-5:TPS78918DBVR
- removed R18: ERA6VEB8200V, Res_820_0p25W:ERA6VEB8200V
- removed U8: MAX682ESA+, C_P_5_MAX682ESA_:MAX682ESA+
- added U10, U4, U9: LD1117S33TR, V_Reg_3.3_SMD:LD1117S33TR
Connections:
- net N$15 renamed AIN3
- net N$17 renamed AIN1
- removed net 3.3: C13.1, C4.2, C5.2, IC2.OUT_2, Q3.G, Q4.G, R1.2, R11.2, R13.2, R14.2, R16.2, R18.2, R2.2, U5.VCC, U6.CSB, U6.VDD, U6.VDDIO, U7.CS, U7.VDD, U7.VDD_IO, U8.!SKIP, U8.IN
- removed net N$14: C3.2, IC2.C2+
- removed net N$18: C3.1, IC2.C2-
- removed net N$19: IC2.FB, IC2.OUT_1
- removed net N$20: C6.2, U8.CXN
- removed net N$22: C6.1, U8.CXP
- removed net N$23: Q1.S, R10.1, U2.SCL
- removed net N$24: R18.1, U8.!SHDN
- removed net N$7 (its old number): C2.2, IC2.C1+
- new net 3.3V: C13.1, IC1.VDD, IC1.VDDH, Q3.G, Q4.G, R11.1, R13.2, R14.2, R16.1, U5.VCC, U6.CSB, U6.VDD, U6.VDDIO, U7.CS, U7.VDD, U7.VDD_IO, U9.OUT
- new net N$25: BT3.-, BT4.+
- new net N$27: BT1.+, S2.2
- new net N$5: Q4.D, R17.1, SPS30.3
- new net SWDCLK: U5.SWDCLK
- new net SWDIO: U5.SWDIO
- net 1.8V: now also R10.1, U10.OUT; no longer C10.2, IC3.OUT, R10.2
- net 5V: now also U4.OUT; no longer C12.1, IC1.VDD, IC1.VDDH, U8.OUT
- net GND: now also U10.GND, U4.GND, U9.GND; no longer BT3.-, C1.2, C10.1, C11.1, C12.2, C4.1, C5.1, IC2.GND_1, IC2.GND_2, IC2.GND_3, IC2.GND_4, IC2.PGND_1, IC2.PGND_2, IC2.PGND_3, IC2.PGND_4, IC3.GND, U8.GND, U8.PGND
- net N$1: no longer IC1.SDA
- net N$12: now also Q1.S, R10.2, U2.SCL; no longer C2.1, IC2.C1-
- net N$2: now also BT1.-; no longer BT1.+, S2.2
- net N$3: now also R1.1, R2.1; no longer IC1.SCL, Q4.D, R17.1, SPS30.3
- net N$4: no longer BT1.-, BT4.+
- net SCL: now also IC1.SCL, R1.2, R11.2, R16.2; no longer R11.1, R16.1, R2.1
- net SDA: now also IC1.SDA, R2.2; no longer R1.1
- net VDD: now also S2.1, U10.IN, U4.IN, U9.IN; no longer C1.1, C11.2, IC2.ENABLE, IC2.IN_1, IC2.IN_2, IC3.!EN, IC3.IN, S2.3
Other:
- note added: "MICS6814"
- note added: "VOLTAGE REGULATOR MESSI A CASO PER ORA ANCORA DA SCEGLIERE"
- note added: "Voltage regulator 1,8V"
- note added: "Voltage regulator 3,3V"
- note added: "Voltage regulator 5V"
- note removed: "AIN1"
- note removed: "AIN3"
- moved on the sheet: BT1, BT2, BT3, BT4, C13, C7, C8, C9, LED2, Q1, Q2, Q3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

Commit message: Inizio PCB
Changed lines of the file:
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@@
 <wire x1="-17.78" y1="208.28" x2="-22.86" y2="208.28" width="0.1524" layer="91"/>
 <junction x="-22.86" y="208.28"/>
-<label x="-40.64" y="205.74" size="1.778" layer="95" rot="R180" xref="yes"/>
+<label x="-33.02" y="205.74" size="1.778" layer="95" rot="R180" xref="yes"/>
 <junction x="-22.86" y="205.74"/>
-<wire x1="-22.86" y1="205.74" x2="-40.64" y2="205.74" width="0.1524" layer="91"/>
+<wire x1="-22.86" y1="205.74" x2="-33.02" y2="205.74" width="0.1524" layer="91"/>
 </segment>
 <segment>
@@
 <wire x1="-22.86" y1="193.04" x2="-22.86" y2="190.5" width="0.1524" layer="91"/>
 <junction x="-22.86" y="190.5"/>
-<label x="-40.64" y="193.04" size="1.778" layer="95" rot="R180" xref="yes"/>
+<label x="-33.02" y="193.04" size="1.778" layer="95" rot="R180" xref="yes"/>
 <junction x="-22.86" y="193.04"/>
-<wire x1="-22.86" y1="193.04" x2="-40.64" y2="193.04" width="0.1524" layer="91"/>
+<wire x1="-22.86" y1="193.04" x2="-33.02" y2="193.04" width="0.1524" layer="91"/>
 </segment>
 <segment>

Commit message: Aggiunto SGP30
Parts:
- removed S2: JS102011SAQN, switch_JS102011SAQN:JS102011SAQN
- added S1: EG1213, switch_TH_HO:EG1213
Connections:
- net N$27: now also S1.2; no longer S2.2
- net VDD: now also S1.1; no longer S2.1
Changed lines of the file:
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@@
 <part name="U1" library="Opamp_SMD" deviceset="TSV912IDT" device=""/>
 <part name="LED2" library="LED_SMD" deviceset="SML-LX1206SRC-TR" device="LED_3P2X1P5_LUM-L"/>
-<part name="S2" library="switch_JS102011SAQN" deviceset="JS102011SAQN" device=""/>
 <part name="C13" library="Condens_10uF" deviceset="CL05A106MP5NUNC" device=""/>
 <part name="GND21" library="supply" deviceset="GND" device=""/>
@@
 <part name="GND25" library="SparkFun-PowerSymbols" deviceset="GND" device=""/>
 <part name="GND27" library="SparkFun-PowerSymbols" deviceset="GND" device=""/>
+<part name="S1" library="switch_TH_HO" deviceset="EG1213" device=""/>
 </parts>
 <sheets>
@@
 <attribute name="NAME" x="-110.3249" y="-2.2652" size="3.48" layer="95" ratio="10" rot="R270"/>
 </instance>
-<instance part="S2" gate="G$1" x="48.26" y="106.68" smashed="yes">
-<attribute name="NAME" x="40.637090625" y="111.761940625" size="1.270490625" layer="95"/>
-<attribute name="VALUE" x="40.631440625" y="101.594290625" size="1.27143125" layer="96"/>
-</instance>
 <instance part="C13" gate="G$1" x="-147.32" y="68.58" smashed="yes" rot="R90">
 <attribute name="NAME" x="-151.13" y="68.58" size="1.778" layer="95" rot="R90"/>
@@
 <attribute name="VALUE" x="91.44" y="9.906" size="1.778" layer="96" align="top-center"/>
 </instance>
+<instance part="S1" gate="G$1" x="48.26" y="106.68" smashed="yes"/>
 </instances>
 <busses>
@@
 <segment>
 <pinref part="BT1" gate="G$1" pin="+"/>
-<pinref part="S2" gate="G$1" pin="2"/>
 <wire x1="66.04" y1="106.68" x2="55.88" y2="106.68" width="0.1524" layer="91"/>
+<pinref part="S1" gate="G$1" pin="2"/>
 </segment>
 </net>
 <net name="VDD" class="0">
 <segment>
-<pinref part="S2" gate="G$1" pin="1"/>
 <wire x1="40.64" y1="109.22" x2="35.56" y2="109.22" width="0.1524" layer="91"/>
 <label x="35.56" y="109.22" size="1.778" layer="95" rot="R180" xref="yes"/>
-</segment>
-<segment>
+<pinref part="S1" gate="G$1" pin="1"/>
+</segment>
+<segment>

Commit message: Aggiunto Voltage Regulators
Parts:
- removed U10, U4, U9: LD1117S33TR, V_Reg_3.3_SMD:LD1117S33TR
- added C1, C2, C3, C4: GRM033C80J104KE15D, Condens_100nF:GRM033C80J104KE15D
- added C5, C6: GRM033R60J105MEA2D, Condens_1uF:GRM033R60J105MEA2D
- added U11: MCP1711T-33I/OTSOT-23-5_OT_MCH, VOLT_REG_3.3_SOT-23-5:MCP1711T-33I/OTSOT-23-5_OT_MCH
- added U12, U8: MC78LC50NTRGTSOT23-5_ONS, VOLT_REG_5V_SOT-23-5:MC78LC50NTRGTSOT23-5_ONS
Connections:
- net 1.8V: now also C6.2, U12.5; no longer U10.OUT
- net 3.3V: now also C2.2, U11.VOUT; no longer U9.OUT
- net 5V: now also C4.2, U8.3; no longer U4.OUT
- net GND: now also C1.1, C2.1, C3.1, C4.1, C5.1, C6.1, U11.GND, U12.2, U8.1; no longer U10.GND, U4.GND, U9.GND
- net VDD: now also C1.2, C3.2, C5.2, U11.!SHDN, U11.VIN, U12.1, U12.3, U8.2; no longer U10.IN, U4.IN, U9.IN

Commit message: Aggiunte capacità 0805
Parts:
- removed C1, C2, C3, C4, C7: GRM033C80J104KE15D, Condens_100nF:GRM033C80J104KE15D
- removed C13: CL05A106MP5NUNC, Condens_10uF:CL05A106MP5NUNC
- removed C5, C6: GRM033R60J105MEA2D, Condens_1uF:GRM033R60J105MEA2D
- removed C8, C9: GRM033R60J103KA01D, Condens_10nF:GRM033R60J103KA01D
- removed LED2: SML-LX1206SRC-TRLED_3P2X1P5_LUM-L, LED_SMD:SML-LX1206SRC-TRLED_3P2X1P5_LUM-L
- removed U11: MCP1711T-33I/OTSOT-23-5_OT_MCH, VOLT_REG_3.3_SOT-23-5:MCP1711T-33I/OTSOT-23-5_OT_MCH
- removed U12: MC78LC50NTRGTSOT23-5_ONS, VOLT_REG_5V_SOT-23-5:MC78LC50NTRGTSOT23-5_ONS
- added C10_10: CL21A226MOQNNNE, Cond_22uF_0805:CL21A226MOQNNNE
- added C1_0.1, C2_0.1, C7_0.01, C8_0.02, C9_0.1: CL21B104KCFNNNE, Cond_100nF_0805:CL21B104KCFNNNE
- added C3_2.2, C4_470P: CL21A475KAQNNNE, Cond_4.7uF_0805:CL21A475KAQNNNE
- added C5_1, C6_2: CL21B105KAFNNNE, Cond_1uF_0805:CL21B105KAFNNNE
- added D1: LTST-C170TBKT, LED_0805:LTST-C170TBKT
- added Q5: MMBT3904-215, BJT_TO-236:MMBT3904-215
- added R29: RNCF0603DTE820R, Res_820OHM:RNCF0603DTE820R
- added V_R_1.8: S-1318D18-M5T1U4, VOLT_REG_1.8_SOT-23-5:S-1318D18-M5T1U4
- added V_R_3.3: MIC5219-3.3YMMMSOP-8LD-PL-1_MCH, Volt_Reg_3.3_8MSOP:MIC5219-3.3YMMMSOP-8LD-PL-1_MCH
- R11: value RNCP0805FTD10K0 -> RP73PF2A130RBTDF; device Res_10K_0p25W:RNCP0805FTD10K0 -> Res_130_0p25:RP73PF2A130RBTDF
- R12: value RNCP0805FTD10K0 -> ERA6VEB8200V; device Res_10K_0p25W:RNCP0805FTD10K0 -> Res_820_0p25W:ERA6VEB8200V
- R13, R14: value RNCP0805FTD10K0 -> RMCF0603FT5M10; device Res_10K_0p25W:RNCP0805FTD10K0 -> Res_5.1MOHM:RMCF0603FT5M10
- R15, R16: value RNCP0805FTD10K0 -> RMCF0603FT10M0; device Res_10K_0p25W:RNCP0805FTD10K0 -> Res_10MOHM_2:RMCF0603FT10M0
- R17: value RNCP0805FTD10K0 -> ERJ-PB6D5101V; device Res_10K_0p25W:RNCP0805FTD10K0 -> Res_5.1K_0805:ERJ-PB6D5101V
- R3, R4: value RMCF0603FT10M0 -> RNCP0805FTD10K0; device Res_10MOHM_2:RMCF0603FT10M0 -> Res_10K_0p25W:RNCP0805FTD10K0
- R5, R6: value RMCF0603FT5M10 -> RNCP0805FTD10K0; device Res_5.1MOHM:RMCF0603FT5M10 -> Res_10K_0p25W:RNCP0805FTD10K0
- R7: value RP73PF2A130RBTDF -> RNCP0805FTD10K0; device Res_130_0p25:RP73PF2A130RBTDF -> Res_10K_0p25W:RNCP0805FTD10K0
- R8: value ERA6VEB8200V -> RNCP0805FTD10K0; device Res_820_0p25W:ERA6VEB8200V -> Res_10K_0p25W:RNCP0805FTD10K0
- R9: value RNCF0603DTE820R -> RNCP0805FTD10K0; device Res_820OHM:RNCF0603DTE820R -> Res_10K_0p25W:RNCP0805FTD10K0
- renumbered U1 to OPAMP, U8 to V_R_5
Connections:
- new net N$14: C4_470P.1, V_R_3.3.BYP
- new net N$15: Q5.B, R17.2
- net 1.8V: now also C6_2.1, C9_0.1.2, R3.1, R5.2, V_R_1.8.VOUT; no longer C6.2, C7.1, R10.1, R12.2, U12.5
- net 3.3V: now also C10_10.2, C3_2.2.1, R10.2, R4.1, R6.2, R8.1, V_R_3.3.OUT; no longer C13.1, C2.2, R11.1, R13.2, R14.2, R16.1, U11.VOUT
- net 5V: now also C2_0.1.1, R11.2, R12.2, R9.2; no longer C4.2, R15.2, R17.2, R8.2
- net AIN1: now also C7_0.01.2, R13.2, R15.2; no longer C8.2, R3.2, R5.2
- net AIN3: now also C8_0.02.1, R14.1, R16.2; no longer C9.2, R4.2, R6.1
- net GND: now also C10_10.1, C1_0.1.2, C2_0.1.2, C3_2.2.2, C4_470P.2, C5_1.2, C6_2.2, C7_0.01.1, C8_0.02.2, C9_0.1.1, R15.1, R16.1, R29.1, V_R_1.8.VSS, V_R_3.3.GND, V_R_3.3.GND_2, V_R_3.3.GND_3, V_R_3.3.GND_4; no longer C1.1, C13.2, C2.1, C3.1, C4.1, C5.1, C6.1, C7.2, C8.1, C9.1, R3.1, R4.1, R9.1, U11.GND, U12.2
- net N$1: now also R9.1; no longer R15.1
- net N$11: now also R12.1; no longer R8.1
- net N$12: now also R3.2; no longer R10.2
- net N$13: now also R11.1; no longer R7.1
- net N$16: now also R5.1; no longer R12.1
- net N$21: now also D1.+; no longer LED2.CATHODE
- net N$5: now also R7.1; no longer R17.1
- net N$7: now also R14.2; no longer R6.2
- net N$8: now also R13.1; no longer R5.1
- net N$9: now also D1.-, R29.2; no longer LED2.ANODE, R9.2
- net SCL: now also R4.2, R8.2; no longer R11.2, R16.2
- net SDA: now also R10.1, R6.1; no longer R13.1, R14.1
- net VDD: now also C1_0.1.1, C5_1.1, V_R_1.8.ON_/_OFF, V_R_1.8.VIN, V_R_3.3.EN, V_R_3.3.IN; no longer C1.2, C3.2, C5.2, U11.!SHDN, U11.VIN, U12.1, U12.3
Other:
- note added: "Serve questa resistenza? Caduta di tensione tra 3 e 3.5 V"
- note added: "VOLTAGE REGULATOR CONTROLLARE LE CONNESSIONI"
- note added: "collegare tra 5V e mics o tra mics e ground?"
- note removed: "VOLTAGE REGULATOR MESSI A CASO PER ORA ANCORA DA SCEGLIERE"
- moved on the sheet: R10, R11, R12, R13, R14, R15, R16, R17, R3, R4, R5, R6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

Commit message: Sistemati nomi su Eagle
Parts:
- removed R29: RNCF0603DTE820R, Res_820OHM:RNCF0603DTE820R
- added R18: ERJ-PB6B3300V, Res_330_0805:ERJ-PB6B3300V
- renumbered D1 to LED1, Q5 to BJT, U2 to SGP30, U5 to MDBT42Q
Connections:
- net GND: now also R18.1; no longer R29.1
- net N$9: now also R18.2; no longer R29.2

Commit message: Aggiunti case 0402
Parts:
- removed C10_10: CL21A226MOQNNNE, Cond_22uF_0805:CL21A226MOQNNNE
- removed C1_0.1, C2_0.1, C7_0.01, C8_0.02, C9_0.1: CL21B104KCFNNNE, Cond_100nF_0805:CL21B104KCFNNNE
- removed C3_2.2, C4_470P: CL21A475KAQNNNE, Cond_4.7uF_0805:CL21A475KAQNNNE
- removed C5_1, C6_2: CL21B105KAFNNNE, Cond_1uF_0805:CL21B105KAFNNNE
- added C1, C10, C11, C12, C13, C2, C3, C4, C5, C6, C7, C8, C9: C0402H102J5GACTU, Condensatore_case_0402:C0402H102J5GACTU
- added PROGRAMMER: BG306-04-A-1-0400-X-X_REVD, Connet_6_BG306-04-A-1-0400-X-X_REVD:BG306-04-A-1-0400-X-X_REVD
- added R19, R20: 8-1879333-9, Resistenza_case_0402:8-1879333-9
- added Y1: ECS-.327-9-16-TR, Crystal-ECS-.327-9-16-TR:ECS-.327-9-16-TR
- R1, R10, R2, R3, R4, R5, R6, R7, R8, R9: value RNCP0805FTD10K0 -> 8-1879333-9; device Res_10K_0p25W:RNCP0805FTD10K0 -> Resistenza_case_0402:8-1879333-9
- R11: value RP73PF2A130RBTDF -> 8-1879333-9; device Res_130_0p25:RP73PF2A130RBTDF -> Resistenza_case_0402:8-1879333-9
- R12: value ERA6VEB8200V -> 8-1879333-9; device Res_820_0p25W:ERA6VEB8200V -> Resistenza_case_0402:8-1879333-9
- R13, R14: value RMCF0603FT5M10 -> 8-1879333-9; device Res_5.1MOHM:RMCF0603FT5M10 -> Resistenza_case_0402:8-1879333-9
- R15, R16: value RMCF0603FT10M0 -> 8-1879333-9; device Res_10MOHM_2:RMCF0603FT10M0 -> Resistenza_case_0402:8-1879333-9
- R17: value ERJ-PB6D5101V -> 8-1879333-9; device Res_5.1K_0805:ERJ-PB6D5101V -> Resistenza_case_0402:8-1879333-9
- R18: value ERJ-PB6B3300V -> 8-1879333-9; device Res_330_0805:ERJ-PB6B3300V -> Resistenza_case_0402:8-1879333-9
- SPS30: value (none) -> BG306-05-A-1-0400-X-X_REVD; device con-lstb:MA05-1 -> Connet_5_BG306-05-A-1-0400-X-X_REVD:BG306-05-A-1-0400-X-X_REVD
Connections:
- net N$1 renamed SDA5
- net N$12 renamed SCL18
- net N$16 renamed SDA18
- removed net N$5: Q4.D, R7.1, SPS30.3
- new net AIN4: C9.1, MDBT42Q.P0.28/AIN4, R19.2, R20.2
- new net N$17: C12.1, MDBT42Q.P0.00/XL1, Y1.2
- new net N$18: C13.1, MDBT42Q.P0.01/XL2, Y1.1
- new net SCL5: Q4.D, R7.2, SPS30.3
- net 1.8V: now also C10.2, C6.1; no longer C6_2.1, C9_0.1.2
- net 3.3V: now also C11.2, C3.1, PROGRAMMER.1; no longer C10_10.2, C3_2.2.1
- net 5V: now also C2.1, R11.1, R12.1, R7.1; no longer C2_0.1.1, R11.2, R12.2, R7.2
- net AIN1: now also C7.2, R13.1, R15.1; no longer C7_0.01.2, R13.2, R15.2
- net AIN3: now also C8.1; no longer C8_0.02.1
- net GND: now also C1.2, C10.1, C11.1, C12.2, C13.2, C2.2, C3.2, C4.2, C5.2, C6.2, C7.1, C8.2, C9.2, PROGRAMMER.4, R15.2, R20.1; no longer C10_10.1, C1_0.1.2, C2_0.1.2, C3_2.2.2, C4_470P.2, C5_1.2, C6_2.2, C7_0.01.1, C8_0.02.2, C9_0.1.1, R15.1
- net N$11: now also R12.2; no longer R12.1
- net N$13: now also R11.2; no longer R11.1
- net N$14: now also C4.1; no longer C4_470P.1
- net N$8: now also R13.2; no longer R13.1
- net SWDCLK: now also PROGRAMMER.3
- net SWDIO: now also PROGRAMMER.2
- net VDD: now also C1.1, C5.1, R19.1; no longer C1_0.1.1, C5_1.1
Other:
- note removed: "Serve questa resistenza? Caduta di tensione tra 3 e 3.5 V"
- moved on the sheet: Q1, Q2, R11, R12, R13, R15, R3, R4, R5, R6, R7

Commit message: Inizio board
Connections:
- new net BJT: BJT.E, OPAMP.VCC+, R11.1, R12.1
- new net P7: MDBT42Q.P0.30AIN6, R17.1
- net 5V: now also BJT.C; no longer OPAMP.VCC+, R11.1, R12.1
Other:
- moved on the sheet: BJT, R17
Changed lines of the file:
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@@
 CONTROLLARE LE CONNESSIONI</text>
 <text x="2.54" y="259.08" size="5.08" layer="91">MICS6814</text>
-<text x="144.78" y="154.94" size="1.778" layer="91">collegare tra 5V e mics o tra mics e ground?</text>
+<text x="93.98" y="246.38" size="1.778" layer="91">collegare tra 5V e mics o tra mics e ground?</text>
 </plain>
 <instances>
@@
 <attribute name="NAME" x="52.07" y="-7.62" size="1.778" layer="95" align="center-left"/>
 </instance>
-<instance part="BJT" gate="G$1" x="132.08" y="154.94" smashed="yes">
-<attribute name="NAME" x="129.54" y="160.02" size="1.778" layer="95"/>
-<attribute name="VALUE" x="132.08" y="144.78" size="1.778" layer="96"/>
+<instance part="BJT" gate="G$1" x="81.28" y="246.38" smashed="yes">
+<attribute name="NAME" x="78.74" y="251.46" size="1.778" layer="95"/>
+<attribute name="VALUE" x="86.36" y="251.46" size="1.778" layer="96"/>
 </instance>
 <instance part="LED1" gate="G$1" x="-104.14" y="-10.16" smashed="yes" rot="R90">
@@
 <attribute name="NAME" x="-30.48148125" y="172.715559375" size="2.54148125" layer="95" rot="R90"/>
 </instance>
-<instance part="R17" gate="G$1" x="116.84" y="154.94" smashed="yes">
-<attribute name="NAME" x="109.215559375" y="157.48148125" size="2.54148125" layer="95"/>
+<instance part="R17" gate="G$1" x="66.04" y="246.38" smashed="yes">
+<attribute name="NAME" x="58.415559375" y="248.92148125" size="2.54148125" layer="95"/>
 </instance>
 <instance part="R18" gate="G$1" x="-104.14" y="-27.94" smashed="yes" rot="R90">
@@
 <net name="5V" class="0">
 <segment>
-<wire x1="96.52" y1="233.68" x2="96.52" y2="226.06" width="0.1524" layer="91"/>
-<label x="96.52" y="233.68" size="1.778" layer="95" xref="yes"/>
-<pinref part="R12" gate="G$1" pin="1"/>
-</segment>
-<segment>
-<pinref part="OPAMP" gate="A" pin="VCC+"/>
-<wire x1="71.12" y1="200.66" x2="73.66" y2="200.66" width="0.1524" layer="91"/>
-<label x="73.66" y="200.66" size="1.778" layer="95" xref="yes"/>
-</segment>
-<segment>
-<wire x1="170.18" y1="187.96" x2="175.26" y2="187.96" width="0.1524" layer="91"/>
-<label x="175.26" y="187.96" size="1.778" layer="95" xref="yes"/>
-<pinref part="R11" gate="G$1" pin="1"/>
-</segment>
-<segment>
 <wire x1="-289.56" y1="175.26" x2="-289.56" y2="177.8" width="0.1524" layer="91"/>
 <label x="-289.56" y="175.26" size="1.778" layer="95" rot="R270" xref="yes"/>
@@
 <pinref part="C2" gate="G$1" pin="1"/>
 <junction x="83.82" y="68.58"/>
+</segment>
+<segment>
+<pinref part="BJT" gate="G$1" pin="C"/>
+<wire x1="83.82" y1="251.46" x2="83.82" y2="256.54" width="0.1524" layer="91"/>
+<label x="83.82" y="256.54" size="1.778" layer="95" rot="R90" xref="yes"/>
 </segment>
 </net>
@@
 <segment>
 <pinref part="BJT" gate="G$1" pin="B"/>
-<wire x1="129.54" y1="154.94" x2="127" y2="154.94" width="0.1524" layer="91"/>
+<wire x1="78.74" y1="246.38" x2="76.2" y2="246.38" width="0.1524" layer="91"/>
 <pinref part="R17" gate="G$1" pin="2"/>
 </segment>
@@
 <segment>
 <pinref part="MDBT42Q" gate="G$1" pin="P0.28/AIN4"/>
-<wire x1="-149.86" y1="25.4" x2="-144.78" y2="25.4" width="0.1524" layer="91"/>
-<wire x1="-144.78" y1="25.4" x2="-144.78" y2="0" width="0.1524" layer="91"/>
-<label x="-144.78" y="0" size="1.778" layer="95" rot="R270" xref="yes"/>
+<wire x1="-149.86" y1="25.4" x2="-142.24" y2="25.4" width="0.1524" layer="91"/>
+<wire x1="-142.24" y1="25.4" x2="-142.24" y2="0" width="0.1524" layer="91"/>
+<label x="-142.24" y="0" size="1.778" layer="95" rot="R270" xref="yes"/>
 </segment>
 </net>
@@
 </segment>
 </net>
+<net name="BJT" class="0">
+<segment>
+<pinref part="BJT" gate="G$1" pin="E"/>
+<wire x1="83.82" y1="241.3" x2="83.82" y2="238.76" width="0.1524" layer="91"/>
+<label x="83.82" y="238.76" size="1.778" layer="95" rot="R270" xref="yes"/>
+</segment>
+<segment>
+<pinref part="R12" gate="G$1" pin="1"/>
+<wire x1="96.52" y1="226.06" x2="96.52" y2="228.6" width="0.1524" layer="91"/>
+<label x="96.52" y="228.6" size="1.778" layer="95" rot="R90" xref="yes"/>
+</segment>
+<segment>
+<pinref part="R11" gate="G$1" pin="1"/>
+<wire x1="170.18" y1="187.96" x2="172.72" y2="187.96" width="0.1524" layer="91"/>
+<label x="172.72" y="187.96" size="1.778" layer="95" xref="yes"/>
+</segment>
+<segment>
+<pinref part="OPAMP" gate="A" pin="VCC+"/>
+<wire x1="71.12" y1="200.66" x2="73.66" y2="200.66" width="0.1524" layer="91"/>
+<label x="73.66" y="200.66" size="1.778" layer="95" xref="yes"/>
+</segment>
+</net>
+<net name="P7" class="0">
+<segment>
+<pinref part="R17" gate="G$1" pin="1"/>
+<wire x1="55.88" y1="246.38" x2="48.26" y2="246.38" width="0.1524" layer="91"/>
+<label x="48.26" y="246.38" size="1.778" layer="95" rot="R180" xref="yes"/>
+</segment>
+<segment>
+<pinref part="MDBT42Q" gate="G$1" pin="P0.30AIN6"/>
+<wire x1="-149.86" y1="20.32" x2="-144.78" y2="20.32" width="0.1524" layer="91"/>
+<wire x1="-144.78" y1="20.32" x2="-144.78" y2="0" width="0.1524" layer="91"/>
+<wire x1="-144.78" y1="0" x2="-152.4" y2="0" width="0.1524" layer="91"/>
+<label x="-152.4" y="0" size="1.778" layer="95" rot="R180" xref="yes"/>
+</segment>
+</net>
