File: PCB_TerzaVersione/circuito_tesi.sch (EAGLE design)
At the start: 57 parts, among them IC1 SCD41-D-R2, J2 S5B-ZR-SM4A-TF_(LF)_(SN)CONN_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, Q1 BSS138, Q2 BSS138, Q3 BSS138, Q4 BSS138, U1 STMICROELECTRONICS_LIS3DHSTMI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, U3 MICS-6814, U6 BME280, Y1 ECS-.327-9-16-TR

Commit message: Tolto resistenze pull up I2C
Parts:
- removed R1, R2: MCS0402MC1002FE000, Res_10K_0402:MCS0402MC1002FE000
Connections:
- net 3.3V: no longer R1.1, R2.1
- net SCL: no longer R1.2
- net SDA: no longer R2.2
Changed lines of the file:
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@@
 <part name="GND11" library="supply" deviceset="GND" device=""/>
 <part name="LED" library="LED_R_LTST-C170KRKT" deviceset="LTST-C170KRKT" device=""/>
-<part name="R1" library="Res_10K_0402" deviceset="MCS0402MC1002FE000" device=""/>
-<part name="R2" library="Res_10K_0402" deviceset="MCS0402MC1002FE000" device=""/>
 <part name="R3" library="Res_10K_0402" deviceset="MCS0402MC1002FE000" device=""/>
 <part name="R4" library="Res_10K_0402" deviceset="MCS0402MC1002FE000" device=""/>
@@
 <attribute name="NAME" x="-209.8086" y="-4.5743" size="1.780009375" layer="95" rot="R90"/>
 </instance>
-<instance part="R1" gate="G$1" x="-228.6" y="22.86" smashed="yes" rot="R90">
-<attribute name="NAME" x="-231.14148125" y="15.235559375" size="2.54148125" layer="95" rot="R90"/>
-</instance>
-<instance part="R2" gate="G$1" x="-215.9" y="22.86" smashed="yes" rot="R90">
-<attribute name="NAME" x="-218.44148125" y="15.235559375" size="2.54148125" layer="95" rot="R90"/>
-</instance>
 <instance part="R3" gate="G$1" x="-350.52" y="25.4" smashed="yes" rot="R90">
 <attribute name="NAME" x="-353.06148125" y="17.775559375" size="2.54148125" layer="95" rot="R90"/>
@@
 <segment>
 <pinref part="MDBT42Q" gate="G$1" pin="P0.08"/>
-<wire x1="-200.66" y1="35.56" x2="-215.9" y2="35.56" width="0.1524" layer="91"/>
-<wire x1="-215.9" y1="35.56" x2="-218.44" y2="35.56" width="0.1524" layer="91"/>
-<wire x1="-215.9" y1="33.02" x2="-215.9" y2="35.56" width="0.1524" layer="91"/>
-<junction x="-215.9" y="35.56"/>
+<wire x1="-200.66" y1="35.56" x2="-218.44" y2="35.56" width="0.1524" layer="91"/>
 <label x="-218.44" y="35.56" size="1.778" layer="95" rot="R180" xref="yes"/>
-<pinref part="R2" gate="G$1" pin="2"/>
 </segment>
 <segment>
@@
 <segment>
 <pinref part="MDBT42Q" gate="G$1" pin="P0.06"/>
-<wire x1="-200.66" y1="40.64" x2="-228.6" y2="40.64" width="0.1524" layer="91"/>
-<wire x1="-228.6" y1="40.64" x2="-233.68" y2="40.64" width="0.1524" layer="91"/>
-<wire x1="-228.6" y1="33.02" x2="-228.6" y2="40.64" width="0.1524" layer="91"/>
-<junction x="-228.6" y="40.64"/>
+<wire x1="-200.66" y1="40.64" x2="-233.68" y2="40.64" width="0.1524" layer="91"/>
 <label x="-233.68" y="40.64" size="1.778" layer="95" rot="R180" xref="yes"/>
-<pinref part="R1" gate="G$1" pin="2"/>
 </segment>
 <segment>
@@
 </segment>
 <segment>
-<wire x1="-228.6" y1="12.7" x2="-228.6" y2="10.16" width="0.1524" layer="91"/>
-<wire x1="-228.6" y1="10.16" x2="-220.98" y2="10.16" width="0.1524" layer="91"/>
-<wire x1="-220.98" y1="10.16" x2="-215.9" y2="10.16" width="0.1524" layer="91"/>
-<wire x1="-215.9" y1="10.16" x2="-215.9" y2="12.7" width="0.1524" layer="91"/>
-<junction x="-220.98" y="10.16"/>
-<wire x1="-220.98" y1="7.62" x2="-220.98" y2="10.16" width="0.1524" layer="91"/>
-<label x="-220.98" y="7.62" size="1.778" layer="95" rot="R270" xref="yes"/>
-<pinref part="R1" gate="G$1" pin="1"/>
-<pinref part="R2" gate="G$1" pin="1"/>
-</segment>
-<segment>

Commit message: Aggiunti nomi
Parts:
- renumbered IC1 to SCD41, J2 to SPS30, PROGRAMMER to PROG, U1 to LIS3DH, U3 to MICS6814, U6 to BME280, V_R_1.8 to VR_1.8, V_R_3.3 to VR_3.3, V_R_5 to VR_5, Y1 to CRYST
