File: PCB_QuartaVersione/PCB.brd (EAGLE design)
At the start: 41 x 41 mm, 55 parts, among them Q1 BSS138, Q2 BSS138, Q3 BSS138, Q4 BSS138

Commit message: Modifiche
Parts:
- moved BME280 0.40 mm to (43.2, 50.1)
- moved S1 0.20 mm to (48.7, 47.1), flipped to the top, turned to 90 degrees
Connections:
- net VDD: now also S1.3; no longer S1.1
Routing:
- net SCL: track 55.4 -> 54.3 mm
- net SDA: track 52.8 -> 52.1 mm
- net GND: vias 34 -> 37

Commit message: Sistemate alcune linee
Parts:
- moved SCD41 0.20 mm to (41.4, 59.4)
Routing:
- net 3.3V: track 139.6 -> 134.5 mm
- net GND: track 7.63 -> 7.44 mm, vias 37 -> 38
