File: PCB_QuartaVersione/PCB.sch (EAGLE design)
At the start: 55 parts, among them Q1 BSS138, Q2 BSS138, Q3 BSS138, Q4 BSS138

Commit message: modifiche per vedere connessione
Parts:
- removed R19, R20: ERJ-2GEJ515X, Res_5,1M_0402:ERJ-2GEJ515X
- added R1, R2: ERJ-2GEJ106X, Res_10M_0402:ERJ-2GEJ106X
Connections:
- net BATTERY: now also R1.1, R2.1; no longer R19.2, R20.2
- net GND: now also R2.2; no longer R20.1
- net VDD: now also R1.2; no longer R19.1
Changed lines of the file:
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@@
 <part name="R13" library="Res_5,1M_0402" deviceset="ERJ-2GEJ515X" device=""/>
 <part name="R14" library="Res_5,1M_0402" deviceset="ERJ-2GEJ515X" device=""/>
-<part name="R19" library="Res_5,1M_0402" deviceset="ERJ-2GEJ515X" device=""/>
-<part name="R20" library="Res_5,1M_0402" deviceset="ERJ-2GEJ515X" device=""/>
 <part name="C1" library="Cond_100n_0402" deviceset="C0402C104K9RACAUTO" device=""/>
 <part name="C2" library="Cond_100n_0402" deviceset="C0402C104K9RACAUTO" device=""/>
@@
 <part name="C12" library="Cond_12p_0402" deviceset="04025A120FAT2A" device=""/>
 <part name="C13" library="Cond_12p_0402" deviceset="04025A120FAT2A" device=""/>
+<part name="R1" library="Res_10M_0402" deviceset="ERJ-2GEJ106X" device=""/>
+<part name="R2" library="Res_10M_0402" deviceset="ERJ-2GEJ106X" device=""/>
 </parts>
 <sheets>
@@
 <attribute name="NAME" x="-5.084440625" y="195.58148125" size="2.54148125" layer="95"/>
 </instance>
-<instance part="R19" gate="G$1" x="35.56" y="-60.96" smashed="yes">
-<attribute name="NAME" x="27.935559375" y="-58.41851875" size="2.54148125" layer="95"/>
-</instance>
-<instance part="R20" gate="G$1" x="53.34" y="-76.2" smashed="yes" rot="R90">
-<attribute name="NAME" x="50.79851875" y="-83.824440625" size="2.54148125" layer="95" rot="R90"/>
-</instance>
 <instance part="C1" gate="G$1" x="48.26" y="66.04" smashed="yes" rot="R90">
 <attribute name="NAME" x="44.45" y="66.04" size="1.778" layer="95" rot="R90"/>
@@
 <instance part="C13" gate="G$1" x="-251.46" y="50.8" smashed="yes">
 <attribute name="NAME" x="-251.46" y="54.61093125" size="1.77843125" layer="95"/>
+</instance>
+<instance part="R1" gate="G$1" x="35.56" y="-60.96" smashed="yes" rot="R180">
+<attribute name="NAME" x="43.184440625" y="-63.50148125" size="2.54148125" layer="95" rot="R180"/>
+</instance>
+<instance part="R2" gate="G$1" x="50.546" y="-76.2" smashed="yes" rot="R270">
+<attribute name="NAME" x="53.08748125" y="-68.575559375" size="2.54148125" layer="95" rot="R270"/>
 </instance>
 </instances>
@@
 <wire x1="60.96" y1="-78.74" x2="60.96" y2="-86.36" width="0.1524" layer="91"/>
 <wire x1="60.96" y1="-86.36" x2="53.34" y2="-86.36" width="0.1524" layer="91"/>
-<pinref part="R20" gate="G$1" pin="1"/>
 <junction x="53.34" y="-86.36"/>
 <pinref part="C9" gate="G$1" pin="2"/>
+<pinref part="R2" gate="G$1" pin="2"/>
+<wire x1="53.34" y1="-86.36" x2="50.546" y2="-86.36" width="0.1524" layer="91"/>
 </segment>
 <segment>
@@
 <wire x1="25.4" y1="-60.96" x2="20.32" y2="-60.96" width="0.1524" layer="91"/>
 <label x="20.32" y="-60.96" size="1.778" layer="95" rot="R180" xref="yes"/>
-<pinref part="R19" gate="G$1" pin="1"/>
+<pinref part="R1" gate="G$1" pin="2"/>
 </segment>
 <segment>
@@
 <wire x1="53.34" y1="-63.5" x2="53.34" y2="-66.04" width="0.1524" layer="91"/>
 <label x="66.04" y="-60.96" size="1.778" layer="95" xref="yes"/>
-<pinref part="R19" gate="G$1" pin="2"/>
-<pinref part="R20" gate="G$1" pin="2"/>
 <pinref part="C9" gate="G$1" pin="1"/>
-</segment>
-</net>
+<pinref part="R2" gate="G$1" pin="1"/>
+<wire x1="53.34" y1="-66.04" x2="50.546" y2="-66.04" width="0.1524" layer="91"/>
+<pinref part="R1" gate="G$1" pin="1"/>
+</segment>
+</net>

Commit message: Aggiunta geolocalizzazione e salvata su file
Parts:
- renumbered R1 to R19, R2 to R20
Changed lines of the file:
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@@
 <part name="C12" library="Cond_12p_0402" deviceset="04025A120FAT2A" device=""/>
 <part name="C13" library="Cond_12p_0402" deviceset="04025A120FAT2A" device=""/>
-<part name="R1" library="Res_10M_0402" deviceset="ERJ-2GEJ106X" device=""/>
-<part name="R2" library="Res_10M_0402" deviceset="ERJ-2GEJ106X" device=""/>
+<part name="R19" library="Res_10M_0402" deviceset="ERJ-2GEJ106X" device=""/>
+<part name="R20" library="Res_10M_0402" deviceset="ERJ-2GEJ106X" device=""/>
 </parts>
 <sheets>
@@
 <attribute name="NAME" x="-251.46" y="54.61093125" size="1.77843125" layer="95"/>
 </instance>
-<instance part="R1" gate="G$1" x="35.56" y="-60.96" smashed="yes" rot="R180">
+<instance part="R19" gate="G$1" x="35.56" y="-60.96" smashed="yes" rot="R180">
 <attribute name="NAME" x="43.184440625" y="-63.50148125" size="2.54148125" layer="95" rot="R180"/>
 </instance>
-<instance part="R2" gate="G$1" x="50.546" y="-76.2" smashed="yes" rot="R270">
-<attribute name="NAME" x="53.08748125" y="-68.575559375" size="2.54148125" layer="95" rot="R270"/>
+<instance part="R20" gate="G$1" x="50.546" y="-76.2" smashed="yes" rot="R270">
+<attribute name="NAME" x="45.46748125" y="-73.655559375" size="2.54148125" layer="95" rot="R270"/>
 </instance>
 </instances>
@@
 <junction x="53.34" y="-86.36"/>
 <pinref part="C9" gate="G$1" pin="2"/>
-<pinref part="R2" gate="G$1" pin="2"/>
+<pinref part="R20" gate="G$1" pin="2"/>
 <wire x1="53.34" y1="-86.36" x2="50.546" y2="-86.36" width="0.1524" layer="91"/>
 </segment>
@@
 <wire x1="25.4" y1="-60.96" x2="20.32" y2="-60.96" width="0.1524" layer="91"/>
 <label x="20.32" y="-60.96" size="1.778" layer="95" rot="R180" xref="yes"/>
-<pinref part="R1" gate="G$1" pin="2"/>
+<pinref part="R19" gate="G$1" pin="2"/>
 </segment>
 <segment>
@@
 <label x="66.04" y="-60.96" size="1.778" layer="95" xref="yes"/>
 <pinref part="C9" gate="G$1" pin="1"/>
-<pinref part="R2" gate="G$1" pin="1"/>
+<pinref part="R20" gate="G$1" pin="1"/>
 <wire x1="53.34" y1="-66.04" x2="50.546" y2="-66.04" width="0.1524" layer="91"/>
-<pinref part="R1" gate="G$1" pin="1"/>
-</segment>
-</net>
+<pinref part="R19" gate="G$1" pin="1"/>
+</segment>
+</net>
