File: PCB/PCB.sch (EAGLE design)
At the start: 55 parts, among them Q1 BSS138, Q2 BSS138, Q3 BSS138, Q4 BSS138

Commit message: Modifiche codice analisi
Other:
- moved on the sheet: BJT, C7, C8, R11, R12, R13, R14, R15, R16, R17
